Commit message: chore(release): prepare v1.3.0 (#83)
- i2rt/robot_models/: version existing arm models and add the YAM Ultra v2 model assets
- i2rt/robots/: add version-aware assembly, recording support, configuration updates, and coverage
- examples/: update MuJoCo, Viser, and minimum-gello workflows for the synchronized APIs
- .agents/, .claude/, .codex/: synchronize URDF and MJCF alignment workflows
- pyproject.toml and uv.lock: synchronize the dev dependency set while retaining package version 1.1.2

Co-authored-by: Codex <noreply@openai.com>

File: i2rt/robot_models/arm/yam_ultra/v1/yam_ultra.urdf (robot description, URDF)
Before this commit: robot yam_ultra, 9 links, 8 joints
Joints:
- removed joint dof_joint1
- removed joint dof_joint2
- removed joint dof_joint3
- removed joint dof_joint4
- removed joint dof_joint5
- removed joint dof_joint6
- removed joint dof_joint7
- removed joint dof_joint8
- added joint joint1: type revolute, parent base, child link1, origin xyz=0 0 0.0733 rpy=0 1.57079632679 3.14159265359, axis -1 0 0, limit lower=-2.61799 upper=3.14159 effort=1 velocity=1
- added joint joint2: type revolute, parent link1, child link2, origin xyz=-0.0455 0.03285 -0.02 rpy=-4.21325e-15 -1.5065e-29 9.98062e-15, axis -3.58252e-15 -1 3.2007e-16, limit lower=0 upper=3.66519 effort=1 velocity=1
- added joint joint3: type revolute, parent link2, child link3, origin xyz=4.08431e-07 -0.0678 0.264 rpy=-6.20015e-15 6.98506e-29 -5.07758e-15, axis 4.54273e-15 1 1.04275e-14, limit lower=0 upper=3.14159 effort=1 velocity=1
- added joint joint4: type revolute, parent link3, child link4, origin xyz=-0.0600003 0.0678 -0.244999 rpy=1.04275e-14 -2.77556e-17 -4.04405e-15, axis 0 1 0, limit lower=-1.69297 upper=1.5708 effort=1 velocity=1
- added joint joint5: type revolute, parent link4, child link5, origin xyz=-0.0403003 -0.0338507 -0.0703851 rpy=-1.02186e-14 2.77556e-17 -6.12323e-17, axis 1 0 0, limit lower=-1.5708 upper=1.5708 effort=1 velocity=1
- added joint joint6: type revolute, parent link5, child gripper, origin xyz=0.0404996 2.39858e-07 -0.0419481 rpy=7.6222e-29 -5.3963e-29 4.42535e-15, axis 1.46014e-15 2.40808e-14 -1, limit lower=-2.0944 upper=2.0944 effort=1 velocity=1
- added joint joint7: type prismatic, parent gripper, child tip_left, origin xyz=0.0239931 -0.0445119 -0.0566919 rpy=-9.48894e-15 -1.66533e-16 3.14159, axis 6.86541e-15 1 0, limit lower=-0.04695 upper=1.84314e-18 effort=1 velocity=1
- added joint joint8: type prismatic, parent gripper, child tip_right, origin xyz=-0.0239931 0.0445119 -0.0566829 rpy=-9.13119e-15 4.4964e-15 -3.14159, axis -6.86541e-15 -1 0, limit lower=-0.04695 upper=8.78204e-18 effort=1 velocity=1
